File: Test.kicad_pcb (KiCad board)
At the start: 4 copper layers, 100 x 50 mm, 199 parts, among them J1 503398-1892, J2 FTSH-107-01-L-DV-K-TR, J3 SFM-115-02-L-D-A-K-TR, J4 0436500300, J5 SFM-115-02-L-D-A-K-TR, J6 0436500300, J7 0436500200, Q2 BSS84, U1 STM32G474RCT6, U2.1 ADM3057EBRWZ, U2.2 ADM3057EBRWZ, U3 ASM330LHHG1TR, U7 LMR33620AQ5RNXTQ1, U8 TPS73733QDRBRQ1, X1 8Mhz

Commit message: test ;
Parts:
- removed C41.1, C41.2: 10uF, STM32_Telemetry_And_IMU_Module:CL05
- added D4.1: LTST-C190KRKT, STM32_Telemetry_And_IMU_Module:LEDC1608X35N, F.Cu at (153.9, 118.0)
- added D4.2: LTST-C190KRKT, STM32_Telemetry_And_IMU_Module:LEDC1608X35N, F.Cu at (153.9, 94.8)
- added FB2.1: 330 Ohms @ 100 MHz, STM32_Telemetry_And_IMU_Module:BLM15EX331SN1D, F.Cu at (157.6, 111.2)
- added FB2.2: 330 Ohms @ 100 MHz, STM32_Telemetry_And_IMU_Module:BLM15EX331SN1D, F.Cu at (157.6, 88.1)
- added FB3.1: 330 Ohms @ 100 MHz, STM32_Telemetry_And_IMU_Module:BLM15EX331SN1D, F.Cu at (155.0, 120.5)
- added FB3.2: 330 Ohms @ 100 MHz, STM32_Telemetry_And_IMU_Module:BLM15EX331SN1D, F.Cu at (155.0, 97.4)
- added FB5.1: 330 Ohms @ 100 MHz, STM32_Telemetry_And_IMU_Module:BLM15EX331SN1D, F.Cu at (155.0, 123.5)
- added FB5.2: 330 Ohms @ 100 MHz, STM32_Telemetry_And_IMU_Module:BLM15EX331SN1D, F.Cu at (155.0, 100.3)
- added FID7: DNP, STM32_Telemetry_And_IMU_Module:FID90X190, B.Cu at (106.5, 127.0)
- added FID8: DNP, STM32_Telemetry_And_IMU_Module:FID90X190, B.Cu at (190.5, 127.0)
- added Q1.1: BSS84, STM32_Telemetry_And_IMU_Module:SOT95P240X120-3N, F.Cu at (157.2, 118.0)
- added Q1.2: BSS84, STM32_Telemetry_And_IMU_Module:SOT95P240X120-3N, F.Cu at (157.2, 94.8)
- added R8.1: 5.1k, STM32_Telemetry_And_IMU_Module:RMCF0402FT, F.Cu at (159.6, 119.5)
- added R8.2: 5.1k, STM32_Telemetry_And_IMU_Module:RMCF0402FT, F.Cu at (159.6, 96.3)
- C14.1, C14.2, C18.1, C18.2: value 10nF -> 47uF; footprint STM32_Telemetry_And_IMU_Module:CL05 -> STM32_Telemetry_And_IMU_Module:CAP_CL32_SAM
- C19.1, C19.2: value 10uF -> 10nF
- C20.1, C20.2: value 100nF -> 10nF
- C21.1, C21.2: value 220nF -> 47uF; footprint STM32_Telemetry_And_IMU_Module:CL05 -> STM32_Telemetry_And_IMU_Module:CAP_CL32_SAM
- FID2: moved to F.Cu
- R7.1, R7.2: value 0 -> 560R
- U2.1, U2.2: value ADM3057EBRWZ -> ISOW1044DFMR; footprint STM32_Telemetry_And_IMU_Module:RW-20_ADI -> STM32_Telemetry_And_IMU_Module:XCVR_ISOW1044BDFMR
- moved FID6 94.8 mm to (190.5, 83.0)
- moved FID2 44.0 mm to (190.5, 83.0), turned to 0 degrees
- moved R7.1 20.0 mm to (153.6, 116.7), turned to 180 degrees
- moved R7.2 20.0 mm to (153.6, 93.6), turned to 180 degrees
- moved C18.1 16.4 mm to (157.5, 122.0)
- moved C18.2 16.4 mm to (157.5, 98.8)
- moved C14.1 16.3 mm to (175.8, 111.2), turned to 180 degrees
- moved C14.2 16.3 mm to (175.8, 88.1), turned to 180 degrees
- moved C20.2 16.3 mm to (173.0, 98.9), turned to 90 degrees
- moved C20.1 16.3 mm to (173.0, 122.0), turned to 90 degrees
- moved FB6.1 12.5 mm to (177.6, 123.5)
- moved FB6.2 12.5 mm to (177.6, 100.3)
- moved C21.1 10.3 mm to (175.1, 122.0), turned to 90 degrees
- moved C21.2 10.3 mm to (175.1, 98.8), turned to 90 degrees
- moved C19.2 9.53 mm to (159.6, 98.9), turned to 90 degrees
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Connections:
- C14.1 pad 1: GND -> ISO_GND.1
- C14.1 pad 2: 3V3 -> ISO_5V.1
- C14.2 pad 1: GND -> ISO_GND.2
- C14.2 pad 2: 3V3 -> ISO_5V.2
- C15.1 pad 2: 3V3 -> NetC15.1_2
- C15.2 pad 2: 3V3 -> NetC15.2_2
- C18.1 pad 1: ISO_GND.1 -> NetC18.1_1
- C18.1 pad 2: ISO_5V.1 -> NetC18.1_2
- C18.2 pad 1: ISO_GND.2 -> NetC18.2_1
- C18.2 pad 2: ISO_5V.2 -> NetC18.2_2
- C19.1 pad 1: GND -> NetC18.1_1
- C19.1 pad 2: 5V -> NetC18.1_2
- C19.2 pad 1: GND -> NetC18.2_1
- C19.2 pad 2: 5V -> NetC18.2_2
- C20.1 pad 1: GND -> NetC20.1_1
- C20.1 pad 2: 5V -> NetC20.1_2
- C20.2 pad 1: GND -> NetC20.2_1
- C20.2 pad 2: 5V -> NetC20.2_2
- C21.1 pad 1: GNDISO.1 -> NetC20.1_1
- C21.1 pad 2: VISOOUT.1 -> NetC20.1_2
- C21.2 pad 1: GNDISO.2 -> NetC20.2_1
- C21.2 pad 2: VISOOUT.2 -> NetC20.2_2
- FB4.1 pad 1: VISOOUT.1 -> NetC20.1_2
- FB4.2 pad 1: VISOOUT.2 -> NetC20.2_2
- FB6.1 pad 1: GNDISO.1 -> NetC20.1_1
- FB6.2 pad 1: GNDISO.2 -> NetC20.2_1
- R7.1 pad 1: NetR7.1_1 -> GND
- R7.1 pad 2: ISO_GND.1 -> NetD4.1_2
- R7.2 pad 1: NetR7.2_1 -> GND
- R7.2 pad 2: ISO_GND.2 -> NetD4.2_2
- U2.1 pad 1: GND -> NetC15.1_2
- U2.1 pad 10: GND -> NetC18.1_1
- U2.1 pad 11: ISO_GND.1 -> NetC20.1_1
- U2.1 pad 12: NetR7.1_1 -> NetC20.1_2
- U2.1 pad 13: CANFD.1_N -> NetC20.1_2
- U2.1 pad 14: CANFD.1_P -> TERM_TOGGLE.1
- U2.1 pad 16: ISO_5V.1 -> ISO_GND.1
- U2.1 pad 17: TERM_TOGGLE.1 -> ISO_GND.1
- U2.1 pad 18: GNDISO.1 -> CANFD.1_N
- U2.1 pad 19: VISOOUT.1 -> CANFD.1_P
- U2.1 pad 2: GND -> CAN_TERM_1
- U2.1 pad 20: GNDISO.1 -> ISO_5V.1
- U2.1 pad 3: 5V -> FDCAN1_TX
- U2.1 pad 4: 3V3 -> FDCAN1_STB
- U2.1 pad 6: (no net) -> GND
- U2.1 pad 7: FDCAN1_TX -> (no net)
- U2.1 pad 8: FDCAN1_STB -> NetQ1.1_1
- U2.1 pad 9: CAN_TERM_1 -> NetC18.1_2
- U2.2 pad 1: GND -> NetC15.2_2
- U2.2 pad 10: GND -> NetC18.2_1
- U2.2 pad 11: ISO_GND.2 -> NetC20.2_1
- U2.2 pad 12: NetR7.2_1 -> NetC20.2_2
- U2.2 pad 13: CANFD.2_N -> NetC20.2_2
- U2.2 pad 14: CANFD.2_P -> TERM_TOGGLE.2
- U2.2 pad 16: ISO_5V.2 -> ISO_GND.2
- U2.2 pad 17: TERM_TOGGLE.2 -> ISO_GND.2
- U2.2 pad 18: GNDISO.2 -> CANFD.2_N
- U2.2 pad 19: VISOOUT.2 -> CANFD.2_P
- U2.2 pad 2: GND -> CAN_TERM_2
- U2.2 pad 20: GNDISO.2 -> ISO_5V.2
- U2.2 pad 3: 5V -> FDCAN2_TX
- U2.2 pad 4: 3V3 -> FDCAN2_STB
- U2.2 pad 6: (no net) -> GND
- U2.2 pad 7: FDCAN2_TX -> (no net)
- U2.2 pad 8: FDCAN2_STB -> NetQ1.2_1
- U2.2 pad 9: CAN_TERM_2 -> NetC18.2_2
Routing:
- net NetC15.2_2: track 0.00 -> 11.6 mm, vias 0 -> 2
- net NetC15.1_2: track 0.00 -> 11.6 mm, vias 0 -> 2
- net NetC20.2_2: track 0.00 -> 9.40 mm
- net NetC20.1_2: track 0.00 -> 9.40 mm
- net CAN_TERM_1: track 26.0 -> 17.2 mm
- net ISO_5V.1: track 8.54 -> 0.84 mm, vias 0 -> 5
- net ISO_5V.2: track 8.49 -> 0.84 mm, vias 0 -> 5
- net TERM_TOGGLE.1: track 8.97 -> 1.85 mm, vias 2 -> 0
- net TERM_TOGGLE.2: track 8.97 -> 1.85 mm, vias 2 -> 0
- net 3V3: track 74.3 -> 67.8 mm
- net NetC20.1_1: track 0.00 -> 6.46 mm
- net NetC20.2_1: track 0.00 -> 6.46 mm
- net NetC18.2_2: track 0.00 -> 6.44 mm
- net NetC18.1_2: track 0.00 -> 6.44 mm
- net NetC18.1_1: track 0.00 -> 6.42 mm
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- added copper zone on F.Cu, net ISO_5V.1
- added copper zone on In2.Cu, net ISO_5V.1
- added copper zone on F.Cu, net ISO_5V.2
- added copper zone on In2.Cu, net ISO_5V.2
- removed copper zone on F.Cu, net GNDISO.1
- removed copper zone on In1.Cu, net GNDISO.1
- removed copper zone on F.Cu, net GNDISO.2
- removed copper zone on In1.Cu, net GNDISO.2
Other:
- rule pad_to_mask_clearance: 0 -> 0.1016
